File: KC1FSZ-Filter-1.kicad_pcb (KiCad board)
At the start: 2 copper layers, 51 x 30 mm, 33 parts, among them J1 Conn_02x05_Odd_Even, J2 Conn_01x03, J3 Conn_01x03, J4 Conn_02x02_Odd_Even, U1 PAT1220-C-6DB, U2 BGA2867, U3 MASW-007221, U4 MASW-007221, U5 BGA2867, U6 PAT1220-C-6DB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

Commit message: Ready for RIT
Parts:
- J4: value Conn_02x02_Odd_Even -> Conn_02x03_Odd_Even; footprint Connector_PinHeader_2.54mm:PinHeader_2x02_P2.54mm_Vertical -> Connector_PinHeader_2.54mm:PinHeader_2x03_P2.54mm_Vertical
- moved J4 2.50 mm to (118.5, 85.0)
Connections:
- C11 pad 1: +5VA -> +5VD
- J4 pad 1: TX_OUT -> +5VD
- J4 pad 3: RX_IN -> TX_OUT
- U5 pad 1: +5VA -> +5VD
Routing:
- net +5VA: track 67.7 -> 21.6 mm
- net +5VD: track 0.00 -> 12.3 mm
